File: cad/spirit-board-v2/ESP32.kicad_sch (KiCad schematic)
At the start: 2 parts, among them J3 Conn_01x12_Pin, J4 Conn_01x02_Pin

Commit message: Out to fab
Parts:
- J3: value Conn_01x12_Pin -> ESP32; footprint (none) -> Connector_PinHeader_2.54mm:PinHeader_1x12_P2.54mm_Vertical
- J4: value Conn_01x02_Pin -> ESP GND
Changed lines of the file:
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@@
   (symbol (lib_id "Connector:Conn_01x12_Pin") (at 111.76 78.74 0) (unit 1)
     (in_bom yes) (on_board yes) (dnp no) (fields_autoplaced)
-    (property "Reference" "J3" (at 112.395 61.595 0)
+    (property "Reference" "J3" (at 112.395 60.96 0)
       (effects (font (size 1.27 1.27)))
     )
-    (property "Value" "Conn_01x12_Pin" (at 112.395 64.135 0)
+    (property "Value" "ESP32" (at 112.395 63.5 0)
       (effects (font (size 1.27 1.27)))
     )
-    (property "Footprint" "" (at 111.76 78.74 0)
+    (property "Footprint" "Connector_PinHeader_2.54mm:PinHeader_1x12_P2.54mm_Vertical" (at 111.76 78.74 0)
       (effects (font (size 1.27 1.27)) hide)
     )
@@
       (effects (font (size 1.27 1.27)))
     )
-    (property "Value" "Conn_01x02_Pin" (at 111.76 46.99 0)
+    (property "Value" "ESP GND" (at 111.76 46.99 0)
       (effects (font (size 1.27 1.27)))
     )
