File: cad/spirit-board-v2/ouija-main.kicad_sch (KiCad schematic)
At the start: 51 parts, among them J5 DEBUG, J6 DEBUG-BACK, J7 UART, SW1 SW_SPST, U2 ATSAMD21J18A-A

Commit message: Out to fab
Parts:
- added C7: 10uF, Capacitor_SMD:C_0805_2012Metric_Pad1.18x1.45mm_HandSolder, symbol Device:C
- C1, C2, C3, C4, C6: footprint Capacitor_SMD:C_1206_3216Metric_Pad1.33x1.80mm_HandSolder -> Capacitor_SMD:C_0805_2012Metric_Pad1.18x1.45mm_HandSolder
- C5: value .1uF -> 1uF; footprint Capacitor_SMD:C_1206_3216Metric_Pad1.33x1.80mm_HandSolder -> Capacitor_SMD:C_0805_2012Metric_Pad1.18x1.45mm_HandSolder
- J5, J6: footprint Connector:Tag-Connect_TC2050-IDC-NL_2x05_P1.27mm_Vertical -> Connector:Tag-Connect_TC2050-IDC-FP_2x05_P1.27mm_Vertical
- J7: footprint (none) -> Connector_PinHeader_2.54mm:PinHeader_1x03_P2.54mm_Vertical
- R1: value R -> 1K
- SW1: value SW_SPST -> SAMD_RST
Connections:
- net 3V3: now also C7.1
- net GND: now also C7.2
- net PWM_IN: now also L10.2, L11.2, L12.2, L13.2, L21.2, L22.2, L23.2, L24.2, L25.2, L26.2, L39.2, L7.2, L8.2, L9.2; no longer L10.1, L11.1, L12.1, L13.1, L21.1, L22.1, L23.1, L24.1, L25.1, L26.1, L39.1, L7.1, L8.1, L9.1
- net at L32.2: now also U2.23 (PB10); no longer U2.6 (PB05)
- net at L15.2: now also U2.12 (PB09); no longer U2.31 (PA14)
- net at U2.43 (PA22): now also L12.1; no longer L23.2
- net at U2.16 (PA07): no longer L8.2
- net at L35.2: now also U2.26 (PB13); no longer U2.11 (PB08)
- net at L19.2: now also U2.2 (PA01); no longer U2.37 (PA18)
- net at U2.42 (PA21): now also L24.1; no longer L22.2
- net at L30.2: now also U2.19 (PA10); no longer U2.64 (PB03)
- net at L3.2: now also U2.5 (PB04); no longer U2.3 (PA02)
- net at L38.2: now also U2.50 (PB23); no longer U2.24 (PB11)
- net at J5.9 (SWDCLK/TCK), J6.9 (SWDCLK/TCK), R1.2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: no longer J5.10 (SWDIO/TMS), J6.10 (SWDIO/TMS), U2.58 (PA31)
- net at U2.44 (PA23): now also L23.1; no longer L24.2
- net at L31.2: now also U2.20 (PA11); no longer U2.5 (PB04)
- net at L14.2: now also U2.37 (PA18); no longer U2.30 (PA13)
- net at L18.2: now also U2.4 (PA03); no longer U2.36 (PA17)
- net at L20.2: now also U2.62 (PB01); no longer U2.38 (PA19)
- net at U2.45 (PA24): now also L11.1; no longer L25.2
- net at U2.25 (PB12): now also L34.2; no longer L39.2
- net at U2.46 (PA25): now also L10.1; no longer L26.2
- net at U2.17 (PA08): now also L28.2; no longer L9.2
- net at U2.35 (PA16): now also L39.1; no longer L17.2
- net at L37.2: now also U2.15 (PA06); no longer U2.23 (PB10)
- net at L16.2: now also U2.10 (PB07); no longer U2.32 (PA15)
- net at L2.2: now also U2.9 (PB06); no longer U2.2 (PA01)
- net at U2.29 (PA12): no longer L13.2
- net at U2.1 (PA00): now also L5.2; no longer L1.2
- net at L36.2: now also U2.27 (PB14); no longer U2.12 (PB09)
- net at U2.13 (PA04): no longer L5.2
- net at U2.14 (PA05): no longer L6.2
- net at U2.18 (PA09): now also L29.2; no longer L10.2
- net at U2.28 (PB15): now also L27.2
- net at L4.2: now also U2.3 (PA02); no longer U2.4 (PA03)
- net at U2.41 (PA20): now also L13.1; no longer L21.2
- net at U2.49 (PB22): now also L22.1
- net at U2.51 (PA27): now also L9.1
- net at U2.53 (PA28): now also L21.1
- net at U2.61 (PB00): now also L8.1; no longer L27.2
- net at U2.63 (PB02): now also L7.1; no longer L29.2
- net at L33.2: now also U2.24 (PB11); no longer U2.9 (PB06)
- new net: J5.10 (SWDIO/TMS), J6.10 (SWDIO/TMS), U2.58 (PA31)
- new net: L25.1, U2.38 (PA19)
- new net: L26.1, U2.36 (PA17)
- new net: L17.2, U2.6 (PB05)
- new net: L1.2, U2.11 (PB08)
- new net: L6.2, U2.64 (PB03)
Other:
- moved on the sheet: J5, J6, J7, L1, L10, L11, L12, L13, L14, L15, L16, L17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
