File: cad/spirit-board-v2/power.kicad_sch (KiCad schematic)
At the start: 2 parts, among them J1 BAT, J2 LIPO RIDE

Commit message: Out to fab
Connections:
- net BAT+: now reaches J1.1 (Pin_1), J2.3 (Pin_3)
Changed lines of the file:
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@@
     (stroke (width 0) (type default))
+  )
+  (label "BAT+" (at 180.34 39.37 0) (fields_autoplaced)
+    (effects (font (size 1.27 1.27)) (justify left bottom))
   )
   (hierarchical_label "5V" (shape input) (at 179.705 81.28 180) (fields_autoplaced)
