File: cad/spirit-board-v2/spirit-board-v2.kicad_pcb (KiCad board)
At the start: 2 copper layers, 355.6 x 170.2 mm, 53 parts, among them J1 BAT, J2 LIPO RIDE, J4 Conn_01x02_Pin, J5 DEBUG, J6 DEBUG-BACK, SW1 SW_SPST, U2 ATSAMD21J18A-A

Commit message: Out to fab
Parts:
- added C7: 10uF, Capacitor_SMD:C_0805_2012Metric_Pad1.18x1.45mm_HandSolder, F.Cu at (267.2, 248.3)
- added J3: ESP32, Connector_PinHeader_2.54mm:PinHeader_1x12_P2.54mm_Vertical, F.Cu at (282.6, 142.2)
- added J7: UART, Connector_PinHeader_2.54mm:PinHeader_1x03_P2.54mm_Vertical, F.Cu at (276.2, 272.4)
- C1, C2, C3, C4, C6: footprint Capacitor_SMD:C_1206_3216Metric_Pad1.33x1.80mm_HandSolder -> Capacitor_SMD:C_0805_2012Metric_Pad1.18x1.45mm_HandSolder
- C5: value .1uF -> 1uF; footprint Capacitor_SMD:C_1206_3216Metric_Pad1.33x1.80mm_HandSolder -> Capacitor_SMD:C_0805_2012Metric_Pad1.18x1.45mm_HandSolder
- J4: value Conn_01x02_Pin -> ESP GND
- J5: footprint Connector:Tag-Connect_TC2050-IDC-NL_2x05_P1.27mm_Vertical -> Connector:Tag-Connect_TC2050-IDC-FP_2x05_P1.27mm_Vertical
- J6: footprint Connector:Tag-Connect_TC2050-IDC-NL_2x05_P1.27mm_Vertical -> Connector:Tag-Connect_TC2050-IDC-FP_2x05_P1.27mm_Vertical; moved to B.Cu
- R1: value R -> 1K
- SW1: value SW_SPST -> SAMD_RST
- moved J2 304.9 mm to (111.1, 198.8), turned to 180 degrees
- moved J1 253.2 mm to (189.9, 142.2), turned to 180 degrees
- moved J4 252.0 mm to (316.9, 142.2), turned to 90 degrees
- moved C5 133.2 mm to (257.8, 245.5), turned to 90 degrees
- moved C6 131.2 mm to (267.2, 252.1)
- moved C1 119.7 mm to (255.3, 245.5), turned to 90 degrees
- moved C3 114.9 mm to (245.3, 256.5), turned to 180 degrees
- moved C2 108.5 mm to (267.0, 261.6)
- moved C4 107.9 mm to (254.0, 267.2), turned to -90 degrees
- moved R1 106.2 mm to (242.6, 274.1), turned to 90 degrees
- moved J5 45.1 mm to (236.2, 269.9)
- moved J6 45.0 mm to (226.7, 280.0), turned to 180 degrees
- moved SW1 21.3 mm to (219.7, 272.4), turned to 180 degrees
- moved U2 14.0 mm to (255.9, 256.5)
- moved L37 11.2 mm to (207.6, 119.6)
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Connections:
- net Net-(J1-Pin_1) renamed /power/BAT+
- J5 pad 10: Net-(J5-SWDCLK/TCK) -> Net-(J5-SWDIO/TMS)
- J6 pad 10: Net-(J5-SWDCLK/TCK) -> Net-(J5-SWDIO/TMS)
- L1 pad 2: Net-(U2-PA00) -> Net-(U2-PB08)
- L10 pad 1: /ESP32/PWM_OUT -> Net-(U2-PA25)
- L10 pad 2: Net-(U2-PA09) -> /ESP32/PWM_OUT
- L11 pad 1: /ESP32/PWM_OUT -> Net-(U2-PA24)
- L11 pad 2: Net-(U2-PA10) -> /ESP32/PWM_OUT
- L12 pad 1: /ESP32/PWM_OUT -> Net-(U2-PA22)
- L12 pad 2: Net-(U2-PA11) -> /ESP32/PWM_OUT
- L13 pad 1: /ESP32/PWM_OUT -> Net-(U2-PA20)
- L13 pad 2: Net-(U2-PA12) -> /ESP32/PWM_OUT
- L14 pad 2: Net-(U2-PA13) -> Net-(U2-PA18)
- L15 pad 2: Net-(U2-PA14) -> Net-(U2-PB09)
- L16 pad 2: Net-(U2-PA15) -> Net-(U2-PB07)
- L17 pad 2: Net-(U2-PA16) -> Net-(U2-PB05)
- L18 pad 2: Net-(U2-PA17) -> Net-(U2-PA03)
- L19 pad 2: Net-(U2-PA18) -> Net-(U2-PA01)
- L2 pad 2: Net-(U2-PA01) -> Net-(U2-PB06)
- L20 pad 2: Net-(U2-PA19) -> Net-(U2-PB01)
- L21 pad 1: /ESP32/PWM_OUT -> Net-(U2-PA28)
- L21 pad 2: Net-(U2-PA20) -> /ESP32/PWM_OUT
- L22 pad 1: /ESP32/PWM_OUT -> Net-(U2-PB22)
- L22 pad 2: Net-(U2-PA21) -> /ESP32/PWM_OUT
- L23 pad 1: /ESP32/PWM_OUT -> Net-(U2-PA23)
- L23 pad 2: Net-(U2-PA22) -> /ESP32/PWM_OUT
- L24 pad 1: /ESP32/PWM_OUT -> Net-(U2-PA21)
- L24 pad 2: Net-(U2-PA23) -> /ESP32/PWM_OUT
- L25 pad 1: /ESP32/PWM_OUT -> Net-(U2-PA19)
- L25 pad 2: Net-(U2-PA24) -> /ESP32/PWM_OUT
- L26 pad 1: /ESP32/PWM_OUT -> Net-(U2-PA17)
- L26 pad 2: Net-(U2-PA25) -> /ESP32/PWM_OUT
- L27 pad 2: Net-(U2-PB00) -> Net-(U2-PB15)
- L28 pad 2: Net-(U2-PB01) -> Net-(U2-PA08)
- L29 pad 2: Net-(U2-PB02) -> Net-(U2-PA09)
- L3 pad 2: Net-(U2-PA02) -> Net-(U2-PB04)
- L30 pad 2: Net-(U2-PB03) -> Net-(U2-PA10)
- L31 pad 2: Net-(U2-PB04) -> Net-(U2-PA11)
- L32 pad 2: Net-(U2-PB05) -> Net-(U2-PB10)
- L33 pad 2: Net-(U2-PB06) -> Net-(U2-PB11)
- L34 pad 2: Net-(U2-PB07) -> Net-(U2-PB12)
- L35 pad 2: Net-(U2-PB08) -> Net-(U2-PB13)
- L36 pad 2: Net-(U2-PB09) -> Net-(U2-PB14)
- L37 pad 2: Net-(U2-PB10) -> Net-(U2-PA06)
- L38 pad 2: Net-(U2-PB11) -> Net-(U2-PB23)
- L39 pad 1: /ESP32/PWM_OUT -> Net-(U2-PA16)
- L39 pad 2: Net-(U2-PB12) -> /ESP32/PWM_OUT
- L4 pad 2: Net-(U2-PA03) -> Net-(U2-PA02)
- L5 pad 2: Net-(U2-PA04) -> Net-(U2-PA00)
- L6 pad 2: Net-(U2-PA05) -> Net-(U2-PB03)
- L7 pad 1: /ESP32/PWM_OUT -> Net-(U2-PB02)
- L7 pad 2: Net-(U2-PA06) -> /ESP32/PWM_OUT
- L8 pad 1: /ESP32/PWM_OUT -> Net-(U2-PB00)
- L8 pad 2: Net-(U2-PA07) -> /ESP32/PWM_OUT
- L9 pad 1: /ESP32/PWM_OUT -> Net-(U2-PA27)
- L9 pad 2: Net-(U2-PA08) -> /ESP32/PWM_OUT
- U2 pad 13: Net-(U2-PA04) -> unconnected-(U2-PA04-Pad13)
- U2 pad 14: Net-(U2-PA05) -> unconnected-(U2-PA05-Pad14)
- U2 pad 16: Net-(U2-PA07) -> unconnected-(U2-PA07-Pad16)
- U2 pad 26: unconnected-(U2-PB13-Pad26) -> Net-(U2-PB13)
- U2 pad 27: unconnected-(U2-PB14-Pad27) -> Net-(U2-PB14)
- U2 pad 28: unconnected-(U2-PB15-Pad28) -> Net-(U2-PB15)
- U2 pad 29: Net-(U2-PA12) -> unconnected-(U2-PA12-Pad29)
- U2 pad 30: Net-(U2-PA13) -> unconnected-(U2-PA13-Pad30)
- U2 pad 31: Net-(U2-PA14) -> unconnected-(U2-PA14-Pad31)
- U2 pad 32: Net-(U2-PA15) -> unconnected-(U2-PA15-Pad32)
- U2 pad 49: unconnected-(U2-PB22-Pad49) -> Net-(U2-PB22)
- U2 pad 50: unconnected-(U2-PB23-Pad50) -> Net-(U2-PB23)
- U2 pad 51: unconnected-(U2-PA27-Pad51) -> Net-(U2-PA27)
- U2 pad 53: unconnected-(U2-PA28-Pad53) -> Net-(U2-PA28)
- U2 pad 58: Net-(J5-SWDCLK/TCK) -> Net-(J5-SWDIO/TMS)
Routing:
- net /ESP32/PWM_OUT: track 0.00 -> 1399.1 mm
- net Net-(U2-PA18): track 0.00 -> 197.0 mm
- net Net-(U2-PA20): track 0.00 -> 164.3 mm
- net Net-(U2-PB23): track 0.00 -> 157.4 mm, vias 0 -> 2
- net Net-(U2-PA17): track 0.00 -> 156.6 mm
- net /ouija-main/3V3: track 0.00 -> 152.3 mm, vias 0 -> 15
- net Net-(U2-PA22): track 0.00 -> 143.3 mm
- net Net-(U2-PB08): track 0.00 -> 140.4 mm
- net Net-(U2-PA19): track 0.00 -> 138.9 mm
- net Net-(U2-PA06): track 0.00 -> 138.1 mm, vias 0 -> 4
- net Net-(U2-PB15): track 0.00 -> 135.4 mm
- net Net-(U2-PB06): track 0.00 -> 119.9 mm
- net /ESP32/ESP_SCL: track 0.00 -> 119.4 mm, vias 0 -> 6
- net /ESP32/ESP_SDA: track 0.00 -> 118.2 mm, vias 0 -> 6
- net Net-(U2-PA24): track 0.00 -> 116.0 mm
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- added copper zone on B.Cu, net /ESP32/ESP_5V5
- added copper zone on F.Cu, net /ouija-main/3V3
- added copper zone on F.Cu, net /power/BAT+
- added copper zone on B.Cu, net GND
Other:
- board size 355.6 x 170.2 mm -> 340.4 x 177.8 mm
- board text added: "OUIJAMATIC"
